File: joystick/gamepad.kicad_pcb (KiCad board)
At the start: 2 copper layers, 112 x 47.6 mm, 40 parts, among them IC1 ATTINY45-S, P2 CONN_01X04, SW1 SW_PUSH, SW2 SW_PUSH, SW3 SW_PUSH, SW4 SW_PUSH, SW5 SW_PUSH, SW6 SW_PUSH, U1 74LS165, U2 74164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

Commit message: Updated joystick's circuit
Parts:
- C1, C2, C3: value C -> 100nF
- C4, C5, C6, C7, C8, C9: value C -> 1uF
- R1: value R -> 10k
- R10, R11, R12, R13, R14, R15, R16, R9: value R -> 120
- R2, R3, R4, R5, R6, R7: value R -> 62k
- R8: value R -> 0
Changed lines of the file:
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@@
     (links 101)
     (no_connects 1)
-    (area 77.165999 89.992999 189.280001 142.220001)
+    (area 77.165999 89.992999 189.280001 137.718001)
     (thickness 1.6)
     (drawings 7)
@@
       (effects (font (size 1 1) (thickness 0.15)))
     )
-    (fp_text value R (at 0 2.1 270) (layer F.Fab)
+    (fp_text value 120 (at 0 2.1 270) (layer F.Fab)
       (effects (font (size 1 1) (thickness 0.15)))
     )
@@
       (effects (font (size 1 1) (thickness 0.15)))
     )
-    (fp_text value R (at 0 2.1 90) (layer F.Fab)
+    (fp_text value 62k (at 0 2.1 90) (layer F.Fab)
       (effects (font (size 1 1) (thickness 0.15)))
     )
@@
       (effects (font (size 1 1) (thickness 0.15)))
     )
-    (fp_text value C (at 0 2.1 270) (layer F.Fab)
+    (fp_text value 1uF (at 0 2.1 270) (layer F.Fab)
       (effects (font (size 1 1) (thickness 0.15)))
     )
@@
       (effects (font (size 1 1) (thickness 0.15)))
     )
-    (fp_text value C (at 0 2.1 270) (layer F.Fab)
+    (fp_text value 100nF (at 0 2.1 270) (layer F.Fab)
       (effects (font (size 1 1) (thickness 0.15)))
     )
@@
       (effects (font (size 1 1) (thickness 0.15)))
     )
-    (fp_text value C (at 0 2.1 90) (layer F.Fab)
+    (fp_text value 100nF (at 0 2.1 90) (layer F.Fab)
       (effects (font (size 1 1) (thickness 0.15)))
     )
@@
       (effects (font (size 1 1) (thickness 0.15)))
     )
-    (fp_text value C (at 0 2.1 90) (layer F.Fab)
+    (fp_text value 1uF (at 0 2.1 90) (layer F.Fab)
       (effects (font (size 1 1) (thickness 0.15)))
     )
@@
       (effects (font (size 1 1) (thickness 0.15)))
     )
-    (fp_text value C (at 0 2.1 270) (layer F.Fab)
+    (fp_text value 1uF (at 0 2.1 270) (layer F.Fab)
       (effects (font (size 1 1) (thickness 0.15)))
     )
@@
       (effects (font (size 1 1) (thickness 0.15)))
     )
-    (fp_text value C (at 0 2.1 90) (layer F.Fab)
+    (fp_text value 1uF (at 0 2.1 90) (layer F.Fab)
       (effects (font (size 1 1) (thickness 0.15)))
     )
@@
       (effects (font (size 1 1) (thickness 0.15)))
     )
-    (fp_text value C (at 0 2.1 270) (layer F.Fab)
+    (fp_text value 1uF (at 0 2.1 270) (layer F.Fab)
       (effects (font (size 1 1) (thickness 0.15)))
     )
@@
       (effects (font (size 1 1) (thickness 0.15)))
     )
-    (fp_text value C (at 0 2.1 90) (layer F.Fab)
+    (fp_text value 1uF (at 0 2.1 90) (layer F.Fab)
       (effects (font (size 1 1) (thickness 0.15)))
     )
@@
       (effects (font (size 1 1) (thickness 0.15)))
     )
-    (fp_text value R (at 0 2.1 270) (layer F.Fab)
+    (fp_text value 10k (at 0 2.1 270) (layer F.Fab)
       (effects (font (size 1 1) (thickness 0.15)))
     )
@@
       (effects (font (size 1 1) (thickness 0.15)))
     )
-    (fp_text value R (at 0 2.1 270) (layer F.Fab)
+    (fp_text value 62k (at 0 2.1 270) (layer F.Fab)
       (effects (font (size 1 1) (thickness 0.15)))
     )
@@
       (effects (font (size 1 1) (thickness 0.15)))
     )
-    (fp_text value R (at 0 2.1 90) (layer F.Fab)
+    (fp_text value 62k (at 0 2.1 90) (layer F.Fab)
       (effects (font (size 1 1) (thickness 0.15)))
     )
@@
       (effects (font (size 1 1) (thickness 0.15)))
     )
-    (fp_text value R (at 0 2.1 270) (layer F.Fab)
+    (fp_text value 62k (at 0 2.1 270) (layer F.Fab)
       (effects (font (size 1 1) (thickness 0.15)))
     )
@@
       (effects (font (size 1 1) (thickness 0.15)))
     )
-    (fp_text value R (at 0 2.1 90) (layer F.Fab)
+    (fp_text value 62k (at 0 2.1 90) (layer F.Fab)
       (effects (font (size 1 1) (thickness 0.15)))
     )
@@
       (effects (font (size 1 1) (thickness 0.15)))
     )
-    (fp_text value R (at 0 2.1 270) (layer F.Fab)
+    (fp_text value 62k (at 0 2.1 270) (layer F.Fab)
       (effects (font (size 1 1) (thickness 0.15)))
     )
@@
       (effects (font (size 1 1) (thickness 0.15)))
     )
-    (fp_text value C (at 0 2.1 270) (layer F.Fab)
+    (fp_text value 100nF (at 0 2.1 270) (layer F.Fab)
       (effects (font (size 1 1) (thickness 0.15)))
     )
@@
       (effects (font (size 1 1) (thickness 0.15)))
     )
-    (fp_text value R (at 0 2.1 180) (layer F.Fab)
+    (fp_text value 0 (at 0 2.1 180) (layer F.Fab)
       (effects (font (size 1 1) (thickness 0.15)))
     )
@@
       (effects (font (size 1 1) (thickness 0.15)))
     )
-    (fp_text value R (at 0 2.1 90) (layer F.Fab)
+    (fp_text value 120 (at 0 2.1 90) (layer F.Fab)
       (effects (font (size 1 1) (thickness 0.15)))
     )
@@
       (effects (font (size 1 1) (thickness 0.15)))
     )
-    (fp_text value R (at 0 2.1 90) (layer F.Fab)
+    (fp_text value 120 (at 0 2.1 90) (layer F.Fab)
       (effects (font (size 1 1) (thickness 0.15)))
     )
@@
       (effects (font (size 1 1) (thickness 0.15)))
     )
-    (fp_text value R (at 0 2.1 270) (layer F.Fab)
+    (fp_text value 120 (at 0 2.1 270) (layer F.Fab)
       (effects (font (size 1 1) (thickness 0.15)))
     )
@@
       (effects (font (size 1 1) (thickness 0.15)))
     )
-    (fp_text value R (at 0 2.1 270) (layer F.Fab)
+    (fp_text value 120 (at 0 2.1 270) (layer F.Fab)
       (effects (font (size 1 1) (thickness 0.15)))
     )
@@
       (effects (font (size 1 1) (thickness 0.15)))
     )
-    (fp_text value R (at 0 2.1 90) (layer F.Fab)
+    (fp_text value 120 (at 0 2.1 90) (layer F.Fab)
       (effects (font (size 1 1) (thickness 0.15)))
     )
@@
       (effects (font (size 1 1) (thickness 0.15)))
     )
-    (fp_text value R (at 0 2.1 90) (layer F.Fab)
+    (fp_text value 120 (at 0 2.1 90) (layer F.Fab)
       (effects (font (size 1 1) (thickness 0.15)))
     )
@@
       (effects (font (size 1 1) (thickness 0.15)))
     )
-    (fp_text value R (at 0 2.1 270) (layer F.Fab)
+    (fp_text value 120 (at 0 2.1 270) (layer F.Fab)
       (effects (font (size 1 1) (thickness 0.15)))
     )
@@
   (segment (start 178.943 112.268) (end 165.608 112.268) (width 0.4) (layer F.Cu) (net 12))
   (segment (start 179.959 111.252) (end 178.943 112.268) (width 0.4) (layer F.Cu) (net 12))
-  (segment (start 157.48 117.315) (end 157.48 114.3) (width 0.4) (layer F.Cu) (net 13) (status 400000))
+  (segment (start 157.48 117.315) (end 157.48 114.3) (width 0.4) (layer F.Cu) (net 13))
   (segment (start 154.94 105.41) (end 156.337 106.807) (width 0.4) (layer F.Cu) (net 13))
   (segment (start 151.13 105.41) (end 154.94 105.41) (width 0.4) (layer F.Cu) (net 13))
@@
   (segment (start 134.7 101.6) (end 137.16 101.6) (width 0.4) (layer F.Cu) (net 28))
   (segment (start 173.482 101.807) (end 173.482 104.267) (width 0.4) (layer F.Cu) (net 32))
-  (segment (start 174.752 109.441) (end 174.752 106.299) (width 0.4) (layer F.Cu) (net 33) (status 400000))
+  (segment (start 174.752 109.441) (end 174.752 106.299) (width 0.4) (layer F.Cu) (net 33))
   (segment (start 174.752 99.314) (end 174.752 106.299) (width 0.4) (layer F.Cu) (net 33))
   (segment (start 174.545 99.107) (end 174.752 99.314) (width 0.4) (layer F.Cu) (net 33))
   (segment (start 174.545 99.107) (end 173.482 99.107) (width 0.4) (layer F.Cu) (net 33))
-  (segment (start 174.752 109.441) (end 174.879 109.568) (width 0.4) (layer F.Cu) (net 33) (status C00000))
+  (segment (start 174.752 109.441) (end 174.879 109.568) (width 0.4) (layer F.Cu) (net 33))
   (segment (start 173.482 99.107) (end 173.482 99.06) (width 0.25) (layer F.Cu) (net 33) (status 30))
   (segment (start 170.942 101.807) (end 170.942 104.267) (width 0.4) (layer F.Cu) (net 34))
@@
   (segment (start 170.942 99.107) (end 170.942 99.06) (width 0.25) (layer F.Cu) (net 35) (status 30))
   (segment (start 173.482 119.507) (end 173.482 121.967) (width 0.4) (layer F.Cu) (net 36))
-  (segment (start 176.149 114.968) (end 176.149 116.459) (width 0.4) (layer F.Cu) (net 37) (status 400000))
+  (segment (start 176.149 114.968) (end 176.149 116.459) (width 0.4) (layer F.Cu) (net 37))
   (segment (start 174.291 124.667) (end 173.482 124.667) (width 0.4) (layer F.Cu) (net 37))
   (segment (start 174.752 117.856) (end 176.149 116.459) (width 0.4) (layer F.Cu) (net 37))
@@
   (segment (start 177.292 99.568) (end 177.292 106.934) (width 0.4) (layer F.Cu) (net 43))
   (segment (start 177.292 106.934) (end 176.149 108.077) (width 0.4) (layer F.Cu) (net 43))
-  (segment (start 176.149 108.077) (end 176.149 109.568) (width 0.4) (layer F.Cu) (net 43) (status 800000))
+  (segment (start 176.149 108.077) (end 176.149 109.568) (width 0.4) (layer F.Cu) (net 43))
   (segment (start 181.102 104.267) (end 181.102 101.807) (width 0.4) (layer F.Cu) (net 44))
   (segment (start 181.102 99.107) (end 180.166 99.107) (width 0.4) (layer F.Cu) (net 45))
