File: joystick/gamepad.sch (KiCad schematic (older format))
At the start: 37 parts, among them IC1 ATTINY45-S, P2 CONN_01X04, SW1 SW_PUSH, SW2 SW_PUSH, SW3 SW_PUSH, SW4 SW_PUSH, SW5 SW_PUSH, SW6 SW_PUSH, U1 74LS165, U2 74164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

Commit message: Fixed hardware bug (74LS14 inputs were left floating) Changed schematics accordingly
Parts:
- added R11, R12, R13, R14, R15, R16: 1k, Resistors_SMD:R_0805_HandSoldering, symbol R
- C1, C2, C3: value C -> 100nF
- C4, C5, C6, C7, C8, C9: value C -> 1uF
- R1: value R -> 10k
- R10: renamed from R13; value R -> 120
- R17: renamed from R2; value R -> 1k
- R18: renamed from R3; value R -> 1k
- R19: renamed from R4; value R -> 1k
- R2: renamed from R12; value R -> 120
- R20: renamed from R5; value R -> 1k
- R21: renamed from R6; value R -> 1k
- R22: renamed from R7; value R -> 1k
- R3: renamed from R16; value R -> 120
- R4: renamed from R11; value R -> 120
- R5: renamed from R15; value R -> 120
- R6: renamed from R10; value R -> 120
- R7: renamed from R14; value R -> 120
- R8: value R -> 0
- R9: value R -> 120
- renumbered P2 to P1
Connections:
- net GND: now also R11.2, R12.2, R13.2, R14.2, R15.2, R16.2
- net at C4.1, R17.2, U3.1: now also R11.1
- net at C5.1, R18.2, U3.3: now also R12.1
- net at C6.1, R19.2, U3.5: now also R13.1
- net at C9.1, R22.2, U3.9: now also R16.1
- net at C7.1, R20.2, U3.13: now also R14.1
- net at C8.1, R21.2, U3.11: now also R15.1
Other:
- moved on the sheet: R17, R18, R19, R20, R21, R22
