File: joystick/pcb/gamepad.kicad_pcb (KiCad board)
At the start: 2 copper layers, 112 x 47.6 mm, 43 parts, among them IC1 ATTINY45-S, P1 CONN_01X04, SW1 SW_PUSH, SW2 SW_PUSH, SW3 SW_PUSH, SW4 SW_PUSH, SW5 SW_PUSH, SW6 SW_PUSH, U1 74LS165, U2 74164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

Commit message: finished firmware small fix in pcb to get buttons in right order TODO: Makefile
Connections:
- U1 pad 12: /B_L -> /B_R
- U1 pad 13: /B_U -> /B_B
- U1 pad 3: /B_R -> /B_U
- U1 pad 4: /B_A -> /B_L
- U1 pad 5: /B_B -> /B_A
- U3 pad 10: /B_A -> /B_L
- U3 pad 12: /B_R -> /B_U
- U3 pad 2: /B_U -> /B_B
- U3 pad 4: /B_L -> /B_R
- U3 pad 8: /B_B -> /B_A
Routing:
- net /B_B: track 24.2 -> 33.6 mm
- net /B_R: track 36.7 -> 29.3 mm
- net /B_A: track 29.3 -> 24.2 mm
- net /B_U: track 33.6 -> 36.7 mm
