File: joystick/pcb/gamepad.sch (KiCad schematic (older format))
At the start: 43 parts, among them IC1 ATTINY45-S, P1 CONN_01X04, SW1 SW_PUSH, SW2 SW_PUSH, SW3 SW_PUSH, SW4 SW_PUSH, SW5 SW_PUSH, SW6 SW_PUSH, U1 74LS165, U2 74164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

Commit message: finished firmware small fix in pcb to get buttons in right order TODO: Makefile
Connections:
- net B_A: now also U1.5 (P6), U3.8; no longer U1.4 (P5), U3.10
- net B_B: now also U1.13 (P2), U3.2; no longer U1.5 (P6), U3.8
- net B_L: now also U1.4 (P5), U3.10; no longer U1.12 (P1), U3.4
- net B_R: now also U1.12 (P1), U3.4; no longer U1.3 (P4), U3.12
- net B_U: now also U1.3 (P4), U3.12; no longer U1.13 (P2), U3.2
Changed lines of the file:
@@
 PB2
 Text Label 6750 1000 0    60   ~ 0
-B_U
+B_B
 Text Label 6750 1650 0    60   ~ 0
-B_L
+B_R
 Text Label 6750 2300 0    60   ~ 0
 B_D
 Text Label 6750 2950 0    60   ~ 0
-B_R
+B_U
 Text Label 6750 3600 0    60   ~ 0
+B_L
+Text Label 6750 4250 0    60   ~ 0
 B_A
-Text Label 6750 4250 0    60   ~ 0
-B_B
 Text Label 6300 1200 0    60   ~ 0
 B_D
 Text Label 6300 1300 0    60   ~ 0
+B_R
+Text Label 6300 1400 0    60   ~ 0
+B_B
+Text Label 6300 1600 0    60   ~ 0
+B_U
+Text Label 6300 1700 0    60   ~ 0
 B_L
-Text Label 6300 1400 0    60   ~ 0
-B_U
-Text Label 6300 1600 0    60   ~ 0
-B_R
-Text Label 6300 1700 0    60   ~ 0
-B_A
 $Comp
 L +5V #PWR011
@@
 	6450 1800 6550 1900
 Text Label 6300 1800 0    60   ~ 0
-B_B
+B_A
 NoConn ~ 6250 1900
 NoConn ~ 6250 1500
